File: EAGLE/Schematic.brd (EAGLE design)
At the start: 80 x 70 mm, 27 parts, among them Q1 IRF520, Y1 16MHz

Commit message: EAGLE: added gerber files
Parts:
- removed 5V: (no value), SparkFun-Connectors:1X03
- removed D1: 1N4007, diode:DO41-10
- removed LED: (no value), adafruit:LED5MM
- added A5-4-3-2, CIOR(ISP): (no value), SparkFun-Connectors:1X04
- added D0-1: (no value), SparkFun-Connectors:1X02
- added D5-6-7, VCC: (no value), SparkFun-Connectors:1X03
- added J1, J2, J3: J5MM, jumper:05
- added PUMP: (no value), adafruit:LED5MM
- moved R2 19.6 mm to (70.2, 35.8), turned to 0 degrees
- moved GND/VCC 12.8 mm to (43.1, 52.1), turned to 270 degrees
- moved LDR 10.4 mm to (3.17, 37.3)
- moved R6 7.49 mm to (5.23, 42.0), turned to 180 degrees
- moved MOISTURE 6.83 mm to (10.0, 49.0), turned to 180 degrees
- moved NOKIA5110TOP 1.41 mm to (43.5, 59.8)
- moved 5V/AUX 1.00 mm to (65.9, 24.6)
- moved GND 0.92 mm to (51.6, 6.81)
- renumbered POWER to 3.3-5V
Connections:
- net 5V: now also J2.1, J2.2, VCC.1, VCC.2, VCC.3; no longer 5V.1, 5V.2, 5V.3
- net A0: now also MOISTURE.3
- net A1: now also LDR.K, R6.2
- net A2: now also A5-4-3-2.1; no longer MOISTURE.1
- net A3: now also A5-4-3-2.2; no longer LDR.K, R6.2
- net A4: now also A5-4-3-2.3
- net A5: now also A5-4-3-2.4
- net D0: now also D0-1.1
- net D1: now also D0-1.2; no longer MODE.1, MODE.2, R5.P$1
- net D10: now also CIOR(ISP).4
- net D11: now also CIOR(ISP).3
- net D12: now also CIOR(ISP).2
- net D13: now also CIOR(ISP).1
- net D2: now also MODE.1, MODE.2, R5.P$1; no longer R4.P$1, SELECT.1, SELECT.2
- net D3: now also R4.P$1, SELECT.1, SELECT.2; no longer NAV.1, NAV.2, R3.P$1
- net D4: now also J1.1, J1.2, NAV.1, NAV.2, R3.P$1
- net D5: now also D5-6-7.1
- net D6: now also D5-6-7.2
- net D7: now also D5-6-7.3
- net D8: now also J3.1, J3.2, PUMP.A; no longer LED.A
- net GND: now also MOISTURE.1; no longer MOISTURE.3
- net N$3: now also PUMP.K; no longer LED.K
- net WP+: no longer D1.A
- net WP-: no longer D1.C
Routing:
- net GND: track 263.4 -> 311.2 mm
- net D4: track 0.00 -> 36.1 mm
- net A1: track 0.00 -> 27.2 mm
- net A0: track 0.00 -> 25.1 mm
- net 5V: track 239.5 -> 262.2 mm
- net A3: track 24.4 -> 4.28 mm
- net D5: track 0.00 -> 12.9 mm
- net D1: track 17.1 -> 4.55 mm
- net D7: track 0.00 -> 11.7 mm
- net D6: track 0.00 -> 11.7 mm
- net A2: track 15.0 -> 4.28 mm
- net WP-: track 27.8 -> 37.2 mm
- net D2: track 18.3 -> 27.6 mm
- net LIGHT: track 15.3 -> 8.55 mm
- net D3: track 24.8 -> 18.2 mm
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Other:
- board size 80 x 70 mm -> 80 x 65 mm
- board text added: "Author: Daniel Nistor"
- board text added: "Water My Plants, v1.1"
- board text added: "Year: 2022"
