File: EAGLE/Schematic.sch (EAGLE design)
At the start: 27 parts, among them Q1 IRF520, Y1 16MHz

Commit message: EAGLE: added gerber files
Parts:
- removed D1: 1N4007, diode:1N4004
- added A5-4-3-2, CIOR(ISP): (no value), SparkFun-Connectors:CONN_04
- added D0-1: (no value), SparkFun-Connectors:CONN_02
- added D5-6-7: (no value), SparkFun-Connectors:CONN_03
- added J1, J2, J3: J5MM, jumper:J5MM
- renumbered 5V to VCC, LED to PUMP, POWER to 3.3-5V
Connections:
- net 5V: now also J2.1, J2.2
- net A0: now also MOISTURE.3
- net A1: now also LDR.C, R6.2
- net A2: now also A5-4-3-2.1; no longer MOISTURE.1
- net A3: now also A5-4-3-2.2; no longer LDR.C, R6.2
- net A4: now also A5-4-3-2.3
- net A5: now also A5-4-3-2.4
- net D0: now also D0-1.1
- net D1: now also D0-1.2; no longer MODE.S, MODE.S1, R5.1
- net D10: now also CIOR(ISP).4
- net D11: now also CIOR(ISP).3
- net D12: now also CIOR(ISP).2
- net D13: now also CIOR(ISP).1
- net D2: now also MODE.S, MODE.S1, R5.1; no longer R4.1, SELECT.S, SELECT.S1
- net D3: now also R4.1, SELECT.S, SELECT.S1; no longer NAV.S, NAV.S1, R3.1
- net D4: now also J1.1, J1.2, NAV.S, NAV.S1, R3.1
- net D5: now also D5-6-7.1
- net D6: now also D5-6-7.2
- net D7: now also D5-6-7.3
- net D8: now also J3.1, J3.2
- net GND: now also MOISTURE.1; no longer MOISTURE.3
- net WP+: no longer D1.A
- net WP-: no longer D1.C
